Commit message: Fix sonar model paths and stabilize CBF startup

File: nps_uw_multibeam_sonar/urdf/multibeam_sonar_blueview_p900.xacro (robot description, xacro)
@@ -11,5 +11,5 @@
       <visual>
         <geometry>
-          <mesh filename="model://blueview_p900_nps_multibeam/meshes/p900.dae" scale="${scale}"/>
+          <mesh filename="file:///home/tb/dave_ws/src/EROAS-main/nps_uw_multibeam_sonar/models/blueview_p900_nps_multibeam_abs/meshes/p900.dae" scale="${scale}"/>
         </geometry>
         <pose xyz="0 0 0" rpy="0 0 0"/>
@@ -17,5 +17,5 @@
       <collision>
         <geometry>
-          <mesh filename="model://blueview_p900_nps_multibeam/meshes/COLLISION-p900.dae" scale="${scale}"/>
+          <mesh filename="file:///home/tb/dave_ws/src/EROAS-main/nps_uw_multibeam_sonar/models/blueview_p900_nps_multibeam_abs/meshes/COLLISION-p900.dae" scale="${scale}"/>
         </geometry>
         <pose xyz="0 0 0" rpy="0 0 0"/>
